File: Microphone.kicad_sch (KiCad schematic)
At the start: 0 parts

Commit message: top-level structure and ESP32-C6 pin assignments nearly sorted
Parts:
- added C10, C11, C9: 1u, Capacitor_SMD:C_1206_3216Metric, symbol Device:C
- added C12, C13: C, Capacitor_SMD:C_0603_1608Metric, symbol Device:C
- added C14, C17, C19: 10u, Capacitor_SMD:CP_Elec_4x5.4, symbol Device:C_Polarized
- added C15, C16, C18, C8: 100n, Capacitor_SMD:C_0603_1608Metric, symbol Device:C
- added C6: 470p, Capacitor_SMD:C_0603_1608Metric, symbol Device:C
- added MK1, MK2: AOM-5024L-HD-F-R, Capacitor_SMD:C_0805_2012Metric, symbol Device:Microphone_Condenser
- added NT1, NT2, NT3: NetTie_2, NetTie:NetTie-2_SMD_Pad0.5mm, symbol Device:NetTie_2
- added R2, R3: 1G, Resistor_SMD:R_0603_1608Metric, symbol Device:R
- added R4, R5, R6, R7: 100, Resistor_SMD:R_0603_1608Metric, symbol Device:R
- added U2: OPA1642AID, Package_SO:SOIC-8_3.9x4.9mm_P1.27mm, symbol Device:Opamp_Dual
- added U7: MIC5205-3.3YM5, Package_TO_SOT_SMD:SOT-23-5, symbol Regulator_Linear:MIC5205-3.3YM5
- added U8: TLV9001IDCK, Package_TO_SOT_SMD:SOT-353_SC-70-5, symbol Amplifier_Operational:TLV9001IDCK
- added U9: PCM1808PWR, Package_SO:TSSOP-14_4.4x5mm_P0.65mm, symbol OpenPolysom:PCM1860DBT
Connections:
- new net: C12.1, R5.1, U2.1, U9.13 (VIN_L)
- new net: C12.2, R5.2, U2.2 (-)
- new net: NT2.1, U9.11 (MD1)
- new net: R4.1, U2.3 (+)
- new net: MK1.2 (+), R2.1, R4.2
- new net: C13.1, R7.1, U2.7, U9.14 (VIN_R)
- new net: C13.2, R7.2, U2.6 (-)
- new net: NT3.1, U9.12 (FMT)
- new net: R6.1, U2.5 (+)
- new net: C6.1, U7.4 (BP)
- new net: NT1.1, U9.10 (MD0)
- new net: MK2.2 (+), R3.1, R6.2
- new net +V: C10.1, C16.1, C17.1, C8.1, U2.8 (V+), U7.5 (OUT), U8.5 (V+), U9.3 (VCC)
- new net BCK: U9.8 (BCK)
- new net DOUT: U9.9 (DOUT)
- new net EN: U7.3 (EN)
- new net LRCK: U9.16 (LRCK)
- new net SCKI: U9.6 (SCKI)
- new net V-: C10.2, C11.2, C14.2, C15.2, C16.2, C17.2, C18.2, C19.2, C6.2, C8.2, C9.2, NT1.2, NT2.2, NT3.2, U2.4 (V-), U7.2 (GND), U8.2 (V-), U9.2 (AGND), U9.5 (DGND)
- new net VBAT: C9.1, U7.1 (IN)
- new net VDD: C18.1, C19.1, U9.4 (VDD)
- new net VREF: C14.1, C15.1, U8.1 (+), U9.1 (VREF)
- new net V_GND: C11.1, MK1.1 (-), MK2.1 (-), R2.2, R3.2, U8.3 (-), U8.4
Other:
- note added: "EN HIGH = Enable (active)"
- note added: "Microphone comparison"
- note added: "Virtual GND = V+/2"
- note added: "https://www.digikey.co.uk/short/hzfn5205"
- company: (none) -> Sunrise designs
- title: (none) -> Open polysomnography board

Commit message: text comments sections added
Other:
- note added: "Ipsum lorem"
- note added: "What's going on here:"
Changed lines of the file:
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@@
 		(company "Sunrise designs")
+	)
+	(text "Ipsum lorem\n"
+		(exclude_from_sim no)
+		(at 18.542 16.256 0)
+		(effects
+			(font
+				(size 1.27 1.27)
+				(color 132 0 0 1)
+			)
+		)
 	)
 	(text "Microphone comparison"
@@
 		)
 	)
+	(text "What's going on here:\n"
+		(exclude_from_sim no)
+		(at 61.468 14.224 0)
+		(effects
+			(font
+				(size 1.905 1.905)
+				(thickness 0.381)
+				(bold yes)
+				(color 132 0 0 1)
+			)
+		)
+	)
 	(junction
 		(at 212.09 46.99)
@@
 	(polyline
 		(pts
+			(xy 12.7 34.29) (xy 118.11 34.29)
+		)
+		(stroke
+			(width 0)
+			(type dash)
+			(color 132 0 0 1)
+		)
+	)
+	(polyline
+		(pts
 			(xy 54.61 82.55) (xy 52.07 81.28)
 		)
@@
 		)
 	)
+	(polyline
+		(pts
+			(xy 118.11 12.7) (xy 118.11 34.29)
+		)
+		(stroke
+			(width 0)
+			(type dash)
+			(color 132 0 0 1)
+		)
+	)

Commit message: some work on sch and docs added
Changed lines of the file:
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@@
+		)
+	)
+	(bus
+		(pts
+			(xy 267.97 76.2) (xy 274.32 76.2)
+		)
+		(stroke
+			(width 0)
+			(type default)
 		)
 	)
@@
 		)
 	)
+	(hierarchical_label "{I2S}"
+		(shape input)
+		(at 274.32 76.2 0)
+		(effects
+			(font
+				(size 1.27 1.27)
+			)
+			(justify left)
+		)
+	)
