File: Polysom.kicad_pcb (KiCad board)
At the start: 2 copper layers, 15 parts, among them J1 Micro_SD_Card, U1 Seeed 113991254, U2 OPA1642AID, U3 ADS1299, U4 LDC1612, U5 LIS2DH12TR

Commit message: some work on sch and docs added
Parts:
- added C10: 1u, Capacitor_SMD:C_1206_3216Metric, F.Cu at (77.1, 125.0)
- added C11: 1u, Capacitor_SMD:C_1206_3216Metric, F.Cu at (77.1, 128.4)
- added C12: C, Capacitor_SMD:C_0603_1608Metric, F.Cu at (56.5, 126.3)
- added C13: C, Capacitor_SMD:C_0603_1608Metric, F.Cu at (56.5, 128.8)
- added C14: 10u, Capacitor_SMD:CP_Elec_4x5.4, F.Cu at (70.4, 122.9)
- added C15: 100n, Capacitor_SMD:C_0603_1608Metric, F.Cu at (56.5, 131.3)
- added C16: 100n, Capacitor_SMD:C_0603_1608Metric, F.Cu at (60.5, 121.3)
- added C17: 10u, Capacitor_SMD:CP_Elec_4x5.4, F.Cu at (70.4, 128.8)
- added C18: 100n, Capacitor_SMD:C_0603_1608Metric, F.Cu at (60.5, 123.8)
- added C19: 10u, Capacitor_SMD:CP_Elec_4x5.4, F.Cu at (70.4, 134.6)
- added C20: 100n, Capacitor_SMD:C_0603_1608Metric, F.Cu at (56.5, 144.3)
- added C21: 1u, Capacitor_SMD:C_1206_3216Metric, F.Cu at (75.9, 144.7)
- added C3: 100n, Capacitor_SMD:C_0603_1608Metric, F.Cu at (75.0, 154.3)
- added C4: 100n, Capacitor_SMD:C_0603_1608Metric, F.Cu at (75.0, 156.8)
- added C5: 10u, Capacitor_SMD:C_0603_1608Metric, F.Cu at (75.0, 159.3)
- added C6: 470p, Capacitor_SMD:C_0603_1608Metric, F.Cu at (56.5, 121.3)
- added C7: 470p, Capacitor_SMD:C_0603_1608Metric, F.Cu at (80.2, 147.7)
- added C8: 100n, Capacitor_SMD:C_0603_1608Metric, F.Cu at (56.5, 123.8)
- added C9: 1u, Capacitor_SMD:C_1206_3216Metric, F.Cu at (77.1, 121.7)
- added FB1: FerriteBead, Inductor_SMD:L_0603_1608Metric, F.Cu at (83.9, 121.3)
- added FB2: FerriteBead, Inductor_SMD:L_0603_1608Metric, F.Cu at (83.9, 123.8)
- added J2: USB_C_Receptacle, Connector_USB:USB_C_Receptacle_HRO_TYPE-C-31-M-12, F.Cu at (64.4, 148.9)
- added MK1: AOM-5024L-HD-F-R, Capacitor_SMD:C_0805_2012Metric, F.Cu at (76.5, 136.2)
- added MK2: AOM-5024L-HD-F-R, Capacitor_SMD:C_0805_2012Metric, F.Cu at (76.5, 139.2)
- added NT1: NetTie_2, NetTie:NetTie-2_SMD_Pad0.5mm, F.Cu at (64.5, 133.3)
- added NT2: NetTie_2, NetTie:NetTie-2_SMD_Pad0.5mm, F.Cu at (64.5, 134.8)
- added NT3: NetTie_2, NetTie:NetTie-2_SMD_Pad0.5mm, F.Cu at (64.5, 136.3)
- added NT4: NetTie_2, NetTie:NetTie-2_SMD_Pad0.5mm, F.Cu at (83.2, 137.4)
- added NT5: NetTie_2, NetTie:NetTie-2_SMD_Pad0.5mm, F.Cu at (80.3, 153.8)
- added NT6: NetTie_2, NetTie:NetTie-2_SMD_Pad0.5mm, F.Cu at (80.3, 155.3)
- added NT7: NetTie_2, NetTie:NetTie-2_SMD_Pad0.5mm, F.Cu at (80.3, 156.8)
- added Q1: 2N7002, Package_TO_SOT_SMD:SOT-23, F.Cu at (88.4, 122.2)
- added Q2: 2N7002, Package_TO_SOT_SMD:SOT-23, F.Cu at (88.4, 126.7)
- added Q3: 2N7002, Package_TO_SOT_SMD:SOT-23, F.Cu at (68.6, 155.8)
- added R10: 10k, Resistor_SMD:R_0603_1608Metric, F.Cu at (83.9, 126.3)
- added R11: 4K7, Resistor_SMD:R_0603_1608Metric, F.Cu at (56.5, 151.8)
- added R12: 4K7, Resistor_SMD:R_0603_1608Metric, F.Cu at (56.5, 154.4)
- added R13: 10k, Resistor_SMD:R_0603_1608Metric, F.Cu at (56.5, 156.9)
- added R14: 10k, Resistor_SMD:R_0603_1608Metric, F.Cu at (56.5, 159.4)
- added R15: 100, Resistor_SMD:R_0603_1608Metric, F.Cu at (83.9, 128.8)
- added R2: 1G, Resistor_SMD:R_0603_1608Metric, F.Cu at (60.5, 126.3)
- added R3: 1G, Resistor_SMD:R_0603_1608Metric, F.Cu at (60.5, 128.8)
- added R4: 100, Resistor_SMD:R_0603_1608Metric, F.Cu at (60.5, 131.3)
- added R5: 100, Resistor_SMD:R_0603_1608Metric, F.Cu at (64.5, 121.3)
- added R6: 100, Resistor_SMD:R_0603_1608Metric, F.Cu at (64.5, 123.8)
- added R7: 100, Resistor_SMD:R_0603_1608Metric, F.Cu at (64.5, 126.3)
- added R8: 10k, Resistor_SMD:R_0603_1608Metric, F.Cu at (56.5, 146.8)
- added R9: 10k, Resistor_SMD:R_0603_1608Metric, F.Cu at (56.5, 149.3)
- added U10: ADS1115IDGS, Package_SO:TSSOP-10_3x3mm_P0.5mm, F.Cu at (85.6, 134.3)
- added U11: MIC5205-3.3YM5, Package_TO_SOT_SMD:SOT-23-5, F.Cu at (75.6, 148.8)
- added U7: MIC5205-3.3YM5, Package_TO_SOT_SMD:SOT-23-5, F.Cu at (76.9, 132.4)
- added U8: TLV9001IDCK, Package_TO_SOT_SMD:SOT-353_SC-70-5, F.Cu at (68.5, 139.4)
- added U9: PCM1808PWR, Package_SO:TSSOP-14_4.4x5mm_P0.65mm, F.Cu at (58.9, 136.0)
- BT1: value Battery_Cell -> 18650
- J1: value Micro_SD_Card -> Micro_SD_Card 693072010801; footprint Connector_Card:microSD_HC_Wuerth_693072010801 -> Connector_Card:microSD_HC_Molex_47219-2001
- L1: value L_Trim -> L_Chest
- U1: value Seeed 113991254 -> ESP32-C6; footprint Seeed:XIAO-ESP32-C6-SMD -> Package_DFN_QFN:QFN-40-1EP_5x5mm_P0.4mm_EP3.6x3.6mm
- moved U1 64.9 mm to (62.2, 160.0)
Connections:
- net Net-(J1-CLK) renamed /ESP-C6/CLK_3
- net Net-(U3-DVDD-Pad48) renamed VBAT
- BT1 pad 1: Net-(BT1-+) -> /ESP-C6/VBAT
- J1 pad 1: unconnected-(J1-DAT2-Pad1) -> /ESP-C6/DAT2
- J1 pad 2: unconnected-(J1-DAT3/CD-Pad2) -> /ESP-C6/CS_3
- J1 pad 3: unconnected-(J1-CMD-Pad3) -> /ESP-C6/MOSI_3
- J1 pad 4: +3V3 -> /ESP-C6/3V3
- J1 pad 6: unconnected-(J1-VSS-Pad6) -> GND
- J1 pad 7: unconnected-(J1-DAT0-Pad7) -> /ESP-C6/MISO_3
- J1 pad 8: unconnected-(J1-DAT1-Pad8) -> /ESP-C6/DAT1
- J1 pad SH: unconnected-(J1-SHIELD-PadSH) -> GND
- R1 pad 2: /RIP/VDD -> +3V3
- U1 pad 10: /ESP-C6/MISO_2 -> unconnected-(U1-MTMS/GPIO4/FSPIHD/ADC1_CH4-Pad10)
- U1 pad 15: (no net) -> unconnected-(U1-GPIO9-Pad15)
- U1 pad 16: (no net) -> unconnected-(U1-GPIO10-Pad16)
- U1 pad 17: (no net) -> unconnected-(U1-GPIO11-Pad17)
- U1 pad 18: (no net) -> unconnected-(U1-GPIO12/USB_D--Pad18)
- U1 pad 19: (no net) -> unconnected-(U1-GPIO13/USB_D+-Pad19)
- U1 pad 2: /ESP-C6/CS_2 -> Net-(U1-VDDA3P3-Pad2)
- U1 pad 20: (no net) -> unconnected-(U1-SPICS0/GPIO24-Pad20)
- U1 pad 21: (no net) -> unconnected-(U1-SPIQ/GPIO25-Pad21)
- U1 pad 22: (no net) -> unconnected-(U1-SPIWP/GPIO26-Pad22)
- U1 pad 23: (no net) -> unconnected-(U1-VDD_SPI/GPIO27-Pad23)
- U1 pad 24: /ESP-C6/MISO_3 -> unconnected-(U1-SPIHD/GPIO28-Pad24)
- U1 pad 3: /ESP-C6/CS_3 -> Net-(U1-VDDA3P3-Pad2)
- U1 pad 4: /ESP-C6/MOSI_2 -> unconnected-(U1-CHIP_PU-Pad4)
- U1 pad 5: /Accelerometer/SDA -> unconnected-(U1-VDDPST1-Pad5)
- U1 pad 6: /Accelerometer/SCL -> Net-(U1-GPIO0/XTAL_32K_P/ADC1_CH0)
- U1 pad 7: unconnected-(U1-GPIO16_D6_TX-Pad7) -> Net-(U1-GPIO1/XTAL_32K_N/ADC1_CH1)
- U1 pad 9: /ESP-C6/SCK_2 -> unconnected-(U1-GPIO3/ADC1_CH3-Pad9)
- U2 pad 1: /Microphone/MIC_OUT_1 -> Net-(U9-VIN_L)
- U2 pad 2: unconnected-(U2A---Pad2) -> Net-(U2A--)
- U2 pad 3: unconnected-(U2A-+-Pad3) -> Net-(U2A-+)
- U2 pad 5: unconnected-(U2B-+-Pad5) -> Net-(U2B-+)
- U2 pad 6: unconnected-(U2B---Pad6) -> Net-(U2B--)
- U2 pad 7: /Microphone/MIC_OUT_2 -> Net-(U9-VIN_R)
- U2 pad 8: /Microphone/V+ -> /Microphone/+V
- U3 pad 19: Net-(U3-AVDD-Pad19) -> /EEG/AVDD
- U3 pad 20: Net-(U3-AVSS-Pad20) -> GND
- U3 pad 21: Net-(U3-AVDD-Pad19) -> /EEG/AVDD
- U3 pad 22: Net-(U3-AVDD-Pad19) -> /EEG/AVDD
- U3 pad 23: Net-(U3-AVSS-Pad20) -> GND
- U3 pad 32: Net-(U3-AVSS-Pad20) -> GND
- U3 pad 33: Net-(U3-DGND-Pad33) -> GND
- U3 pad 34: unconnected-(U3-DIN-Pad34) -> /MOSI
- U3 pad 39: unconnected-(U3-~{CS}-Pad39) -> /CS
- U3 pad 40: unconnected-(U3-SCLK-Pad40) -> /SCK
- U3 pad 43: unconnected-(U3-DOUT-Pad43) -> /MISO
- U3 pad 49: Net-(U3-DGND-Pad33) -> GND
- U3 pad 51: Net-(U3-DGND-Pad33) -> GND
- U3 pad 53: unconnected-(U3-AVSS1-Pad53) -> GND
- U3 pad 54: unconnected-(U3-AVDD1-Pad54) -> /EEG/AVDD
- U3 pad 56: Net-(U3-AVDD-Pad19) -> /EEG/AVDD
- U3 pad 57: Net-(U3-AVSS-Pad20) -> GND
- U3 pad 58: Net-(U3-AVSS-Pad20) -> GND
- U3 pad 59: Net-(U3-AVDD-Pad19) -> /EEG/AVDD
- U4 pad 13: /RIP/GND -> GND
- U4 pad 3: /RIP/GND -> GND
- U4 pad 6: /RIP/SD -> /SHDN
- U4 pad 7: /RIP/VDD -> +3V3
- U4 pad 8: /RIP/GND -> GND
- U5 pad 10: Net-(U5-GND-Pad10) -> GND
- U5 pad 11: Net-(U5-GND-Pad10) -> GND
- U5 pad 12: Net-(U5-GND-Pad10) -> GND
- U5 pad 13: Net-(U5-GND-Pad10) -> GND
- U5 pad 14: Net-(U5-GND-Pad10) -> GND
- U5 pad 3: unconnected-(U5-SDO-Pad3) -> GND
- U5 pad 7: unconnected-(U5-Vdd_IO-Pad7) -> +3V3
- U5 pad 8: unconnected-(U5-Vdd-Pad8) -> +3V3
- U5 pad 9: Net-(U5-GND-Pad10) -> GND
